File: hardware/color-v2.kicad_pcb (KiCad board)
At the start: 2 copper layers, 25 x 20 mm, 30 parts, among them P1 CON-SENSOR2, P2 DEBUG, P3 BOOT, Q1 2N7002P, U1 TCS3472, U2 XMC1300, U3 DRILL, U4 DRILL, U5 DRILL, U6 DRILL

Commit message: Data Cleanup
Parts:
- moved U2 0.09 mm to (105.1, 79.6)
Routing:
- net SDA: track 14.0 -> 13.1 mm
- net Net-(D1-Pad1): track 2.59 -> 1.94 mm
- net Net-(P3-Pad2): track 1.88 -> 1.33 mm
- net VCC: track 57.8 -> 57.2 mm
Other:
- net class Default removed
- board text added: "Copyright Tinkerforge GmbH 2023. This documentation describes Open Hardware and is licensed under the CERN OHL v. 1.1. You may redistribute and modify this documentation under the terms of the CERN OHL v.1.1. (http://ohwr.org/cernohl). This documentation is distributed WITHOUT ANY EXPRESS OR IMPLIED WARRANTY, INCLUDING OF MERCHANTABILITY, SATISFACTORY QUALITY AND FITNESS FOR A PARTICULAR PURPOSE.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"
- board text removed: "Copyright Tinkerforge GmbH 2018. This documentation describes Open Hardware and is licensed under the CERN OHL v. 1.1. You may redistribute and modify this documentation under the terms of the CERN OHL v.1.1. (http://ohwr.org/cernohl). This documentation is distributed WITHOUT ANY EXPRESS OR IMPLIED WARRANTY, INCLUDING OF MERCHANTABILITY, SATISFACTORY QUALITY AND FITNESS FOR A PARTICULAR PURPOSE.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"
